Commit message: Add Yonsoku robot configuration and sensor files
- Introduced yonsoku_robot_physics.usd to define the physical properties of the Yonsoku robot.
- Added yonsoku_robot_sensor.usd to specify the sensor configurations for the Yonsoku robot.
- Created yonsoku_robot.usd to integrate the robot's physics and sensor configurations into a single USD file.

File: source/isaaclab_rl_experiments/isaaclab_rl_experiments/assets/robots/yonsoku/urdf/yonsoku_robot.urdf (robot description, URDF)
Before this commit: robot yonsoku_robot, 19 links, 18 joints
Links:
- link LB1: geometry collision mesh filename=../meshes/lb_hip.stl scale=0.002 0.002 0.002; visual mesh filename=../meshes/lb_hip.stl
- link LB2: geometry collision mesh filename=../meshes/l_upper_leg.stl; visual mesh filename=../meshes/l_upper_leg.stl
- link LB3: geometry collision mesh filename=../meshes/lower_leg.stl; visual mesh filename=../meshes/lower_leg.stl
- link LF1: geometry collision mesh filename=../meshes/lf_hip.stl scale=0.002 0.002 0.002; visual mesh filename=../meshes/lf_hip.stl
- link LF2: geometry collision mesh filename=../meshes/l_upper_leg.stl; visual mesh filename=../meshes/l_upper_leg.stl
- link LF3: geometry collision mesh filename=../meshes/lower_leg.stl; visual mesh filename=../meshes/lower_leg.stl
- link RB1: geometry collision mesh filename=../meshes/rb_hip.stl scale=0.002 0.002 0.002; visual mesh filename=../meshes/rb_hip.stl
- link RB2: geometry collision mesh filename=../meshes/r_upper_leg.stl; visual mesh filename=../meshes/r_upper_leg.stl
- link RB3: geometry collision mesh filename=../meshes/lower_leg.stl; visual mesh filename=../meshes/lower_leg.stl
- link RF1: geometry collision mesh filename=../meshes/rf_hip.stl scale=0.002 0.002 0.002; visual mesh filename=../meshes/rf_hip.stl
- link RF2: geometry collision mesh filename=../meshes/r_upper_leg.stl; visual mesh filename=../meshes/r_upper_leg.stl
- link RF3: geometry collision mesh filename=../meshes/lower_leg.stl; visual mesh filename=../meshes/lower_leg.stl
- link body_link: geometry collision mesh filename=../meshes/base.stl scale=0.001 0.001 0.001; visual mesh filename=../meshes/base.stl scale=0.001 0.001 0.001
